File: leapbot.sch (KiCad schematic (older format))
At the start: 97 parts, among them J1 629105150521, J2 Conn_01x04_Male, J3 BM06B-SRSS-TB, J4 BM06B-SRSS-TB, Q1 FDV301N, Q2 FDV301N, SW1 1825910-6, SW2 1825910-6, U1 QRE1113GR, U10 DRV8872DDA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

Commit message: Add silkscreen annotations and logo, update titleblocks
Parts:
- added SYM1: LOGO, leapbot:logo, symbol Graphic:SYM_Arrow45_Large
- U4: PartNumber (none) -> ADP2302ARDZ-3.3
Changed lines of the file:
@@
 encoding utf-8
 Sheet 1 1
-Title ""
-Date ""
-Rev ""
-Comp ""
-Comment1 ""
+Title "Leapbot"
+Date "2020-05-29"
+Rev "0.0.0"
+Comp "Leetware"
+Comment1 "github.com/hoani/leap-bot"
 Comment2 ""
 Comment3 ""
@@
 Wire Wire Line
 	6850 5000 6950 5000
-Text Notes 9600 5850 0    50   ~ 0
+Text Notes 9850 5900 0    50   ~ 0
 Extras: \n- 2x Motor/Encoder Cable, 50mm, 6-pin\n   A06SR06SR30K51B\n- 1x Magnetic encoder pair Polou 4761\n   2183-4761-ND\n- 2x Pololu Motor 2217\n   2183-2217-ND\n- wheels: https://www.aliexpress.com/item/32854636812.html
 Wire Wire Line
@@
 F 2 "Package_SO:SOIC-8-1EP_3.9x4.9mm_P1.27mm_EP2.29x3mm" H 2650 3850 50  0001 L CNN
 F 3 "https://www.analog.com/media/en/technical-documentation/data-sheets/ADP2302_2303.pdf" H 2300 4800 50  0001 C CNN
+F 4 "ADP2302ARDZ-3.3" H 2500 4200 50  0001 C CNN "PartNumber"
 	1    2500 4200
 	1    0    0    -1
@@
 Wire Wire Line
 	6850 3000 6950 3000
+$Comp
+L Graphic:SYM_Arrow45_Large SYM1
+U 1 1 5FD413E8
+P 10700 3900
+F 0 "SYM1" H 10700 4060 50  0001 C CNN
+F 1 "LOGO" H 10838 3899 50  0000 L CNN
+F 2 "leapbot:logo" H 10700 3900 50  0001 C CNN
+F 3 "~" H 10700 3900 50  0001 C CNN
+	1    10700 3900
+	1    0    0    -1
+$EndComp
 $EndSCHEMATC

Commit message: Add billofmaterials
Other:
- note removed: "Extras: \n- 2x Motor/Encoder Cable, 50mm, 6-pin\n A06SR06SR30K51B\n- 1x Magnetic encoder pair Polou 4761\n 2183-4761-ND\n- 2x Pololu Motor 2217\n 2183-2217-ND\n- wheels: https://www.aliexpress.com/item/32854636812.html"
Changed lines of the file:
@@
 Wire Wire Line
 	6850 5000 6950 5000
-Text Notes 9850 5900 0    50   ~ 0
-Extras: \n- 2x Motor/Encoder Cable, 50mm, 6-pin\n   A06SR06SR30K51B\n- 1x Magnetic encoder pair Polou 4761\n   2183-4761-ND\n- 2x Pololu Motor 2217\n   2183-2217-ND\n- wheels: https://www.aliexpress.com/item/32854636812.html
 Wire Wire Line
 	800  3800 800  3700

Commit message: Corrected some ADC assignments
Connections:
- wire segments 262 -> 263
Changed lines of the file:
@@
 Text Label 7100 1250 0    50   ~ 0
 BOOT_OP
-NoConn ~ 5650 3000
 NoConn ~ 5650 3100
 $Comp
@@
 Text Label 6750 6000 0    50   ~ 0
 LS_PF
-Text Label 5400 4100 0    50   ~ 0
+Text Label 6950 3700 0    50   ~ 0
 LS_FF
-Text Label 5400 4500 0    50   ~ 0
+Text Label 6950 3500 0    50   ~ 0
 LS_FL
-Text Label 6950 4300 0    50   ~ 0
+Text Label 5400 3000 0    50   ~ 0
 LS_FR
-Text Label 6950 4100 0    50   ~ 0
+Text Label 6950 3200 0    50   ~ 0
 LS_BR
-Text Label 5400 4200 0    50   ~ 0
+Text Label 6950 3400 0    50   ~ 0
 LS_BL
-Text Label 6950 3300 0    50   ~ 0
+Text Label 6950 3000 0    50   ~ 0
 LS_BB
 Text Label 6950 4900 0    50   ~ 0
@@
 Text Label 6950 3600 0    50   ~ 0
 M1_EB
-Text Label 6950 3500 0    50   ~ 0
+Text Label 6950 4100 0    50   ~ 0
 M2_EA
-Text Label 6950 3400 0    50   ~ 0
+Text Label 6950 4000 0    50   ~ 0
 M2_EB
 $Comp
@@
 Wire Wire Line
 	2000 5950 2400 5950
-Text Label 6950 3000 0    50   ~ 0
+Text Label 5400 4000 0    50   ~ 0
 LS_PF
-Text Label 6950 3200 0    50   ~ 0
+Text Label 5400 4100 0    50   ~ 0
 LS_PB
 Text Label 6950 4600 0    50   ~ 0
@@
 Text Label 1500 7450 0    50   ~ 0
 LED7
-Text Label 6950 3700 0    50   ~ 0
+Text Label 5400 4400 0    50   ~ 0
 LED0
-Text Label 5400 4300 0    50   ~ 0
+Text Label 5400 4200 0    50   ~ 0
 LED1
-Text Label 6950 4000 0    50   ~ 0
+Text Label 6950 4300 0    50   ~ 0
 LED2
 Text Label 6950 3800 0    50   ~ 0
 LED3
-Text Label 5400 4000 0    50   ~ 0
+Text Label 5400 4500 0    50   ~ 0
 LED4
-Text Label 5400 4400 0    50   ~ 0
+Text Label 5400 4300 0    50   ~ 0
 LED5
 Text Label 6950 4200 0    50   ~ 0
@@
 	1    0    0    -1
 $EndComp
+Wire Wire Line
+	5400 3000 5650 3000
+NoConn ~ 6950 3300
 $EndSCHEMATC
